File: two_terminal_current_source/two_terminal_current_source.kicad_pcb (KiCad board)
At the start: 2 copper layers, 12.1 x 31 mm, 19 parts, among them Q1 MMBT3904, Q2 MMBT3906, Q3 MMBT3904, U1 TL431DBZ, U2 LM358

Commit message: Move connectors, fix silkscreen, add identifier
* Move output to left side to suit mechanical enclosure
* Move sense resistor input pads to side of board to suit mechanical enclosure
* Move more component identifiers to silkscreen layer
* Add board version, identification
Parts:
- removed R2: 800, Connector_PinHeader_2.54mm:PinHeader_1x02_P2.54mm_Vertical
- added TP4: RsA, Connector_PinHeader_2.54mm:PinHeader_1x01_P2.54mm_Vertical, F.Cu at (107.3, 95.2)
- added TP5: RsB, Connector_PinHeader_2.54mm:PinHeader_1x01_P2.54mm_Vertical, F.Cu at (99.1, 95.2)
- moved TP2 5.39 mm to (99.1, 72.4)
- moved Q2 1.27 mm to (102.9, 72.3), turned to 180 degrees
- moved C2 1.14 mm to (107.3, 71.4)
- moved R4 1.14 mm to (107.3, 73.2)
Routing:
- net GND: track 24.3 -> 33.0 mm
- net Net-(Q2-Pad2): track 10.4 -> 11.9 mm
- net Net-(Q2-Pad3): track 3.91 -> 2.35 mm
- net +12V: track 27.9 -> 26.6 mm
- net Net-(Q2-Pad1): track 5.23 -> 5.96 mm
Other:
- board text added: "r2i v2"
- board text added: "thouters"
